File: PCB/Estebquencer/Estebquencer.sch (KiCad schematic (older format))
At the start: 1 part

Commit message: nuevo cambio
Parts:
- added IC2: DAC7513_DCN, symbol DAC7513_DCN
- added R1, R2, R3, R4: 10Kb, symbol POT
- gave numbers to parts that had none: 1
Connections:
- new net +3V3: R1.1, R2.1, R3.1, R4.1
- new net Audio_Out: IC2.1 (VOUT), IC2.2 (VFB)
- new net Earth: R1.3, R2.3, R3.3, R4.3
- new net Pot_1: R1.2
- new net Pot_2: R2.2
- new net Pot_3: R3.2
- new net Pot_4: R4.2
Other:
- moved on the sheet: IC1
Changed lines of the file:
@@
 LIBS:valves
 LIBS:libreria_proyecto
+LIBS:Estebquencer-cache
 EELAYER 26 0
 EELAYER END
@@
 $EndDescr
 $Comp
-L STM32F103C8T6 U?
+L STM32F103C8T6 IC1
 U 1 1 58712984
-P 3950 3150
-F 0 "U?" H 3950 5218 50  0000 C CNN
-F 1 "STM32F103C8T6" H 3950 5127 50  0000 C CNN
-F 2 "LQFP48" H 3950 5036 50  0000 C CNN
-F 3 "" H 3950 3150 50  0000 C CNN
-	1    3950 3150
+P 4750 2950
+F 0 "IC1" H 4750 5018 50  0000 C CNN
+F 1 "STM32F103C8T6" H 4750 4927 50  0000 C CNN
+F 2 "LQFP48" H 4750 4836 50  0000 C CNN
+F 3 "" H 4750 2950 50  0000 C CNN
+	1    4750 2950
 	1    0    0    -1
 $EndComp
+$Comp
+L DAC7513_DCN IC2
+U 1 1 5871366C
+P 9350 1500
+F 0 "IC2" H 9350 2178 50  0000 C CNN
+F 1 "DAC7513_DCN" H 9350 2087 50  0000 C CNN
+F 2 "" H 9400 1100 50  0000 L CNN
+F 3 "" H 9350 1500 50  0000 C CNN
+	1    9350 1500
+	1    0    0    -1
+$EndComp
+Text GLabel 10450 1300 2    60   Input ~ 0
+Audio_Out
+Wire Wire Line
+	9950 1300 10250 1300
+Wire Wire Line
+	10250 1300 10450 1300
+Wire Wire Line
+	9950 1500 10250 1500
+Wire Wire Line
+	10250 1500 10250 1300
+Connection ~ 10250 1300
+$Comp
+L POT R1
+U 1 1 58713A3D
+P 1350 6400
+F 0 "R1" H 1280 6446 50  0000 R CNN
+F 1 "10Kb" H 1280 6355 50  0000 R CNN
+F 2 "" H 1350 6400 50  0000 C CNN
+F 3 "" H 1350 6400 50  0000 C CNN
+	1    1350 6400
+	1    0    0    -1
+$EndComp
+Text GLabel 1650 6400 2    60   Input ~ 0
+Pot_1
+Wire Wire Line
+	1650 6400 1500 6400
+$Comp
+L Earth #PWR?
+U 1 1 58713CAC
+P 1350 6700
+F 0 "#PWR?" H 1350 6450 50  0001 C CNN
+F 1 "Earth" H 1350 6550 50  0001 C CNN
+F 2 "" H 1350 6700 50  0000 C CNN
+F 3 "" H 1350 6700 50  0000 C CNN
+	1    1350 6700
+	1    0    0    -1
+$EndComp
+Wire Wire Line
+	1350 6550 1350 6700
+Text GLabel 1350 6050 1    60   Input ~ 0
++3V3
+Wire Wire Line
+	1350 6250 1350 6050
+$Comp
+L POT R2
+U 1 1 58713D88
+P 2400 6400
+F 0 "R2" H 2330 6446 50  0000 R CNN
+F 1 "10Kb" H 2330 6355 50  0000 R CNN
+F 2 "" H 2400 6400 50  0000 C CNN
+F 3 "" H 2400 6400 50  0000 C CNN
+	1    2400 6400
+	1    0    0    -1
+$EndComp
+Text GLabel 2700 6400 2    60   Input ~ 0
+Pot_2
+Wire Wire Line
+	2700 6400 2550 6400
+$Comp
+L Earth #PWR?
+U 1 1 58713D90
+P 2400 6700
+F 0 "#PWR?" H 2400 6450 50  0001 C CNN
+F 1 "Earth" H 2400 6550 50  0001 C CNN
+F 2 "" H 2400 6700 50  0000 C CNN
+F 3 "" H 2400 6700 50  0000 C CNN
+	1    2400 6700
+	1    0    0    -1
+$EndComp
+Wire Wire Line
+	2400 6550 2400 6700
+Text GLabel 2400 6050 1    60   Input ~ 0
++3V3
+Wire Wire Line
+	2400 6250 2400 6050
+$Comp
+L POT R3
+U 1 1 58713E04
+P 3450 6400
+F 0 "R3" H 3380 6446 50  0000 R CNN
+F 1 "10Kb" H 3380 6355 50  0000 R CNN
+F 2 "" H 3450 6400 50  0000 C CNN
+F 3 "" H 3450 6400 50  0000 C CNN
+	1    3450 6400
+	1    0    0    -1
+$EndComp
+Text GLabel 3750 6400 2    60   Input ~ 0
+Pot_3
+Wire Wire Line
+	3750 6400 3600 6400
+$Comp
+L Earth #PWR?
+U 1 1 58713E0C
+P 3450 6700
+F 0 "#PWR?" H 3450 6450 50  0001 C CNN
+F 1 "Earth" H 3450 6550 50  0001 C CNN
+F 2 "" H 3450 6700 50  0000 C CNN
+F 3 "" H 3450 6700 50  0000 C CNN
+	1    3450 6700
+	1    0    0    -1
+$EndComp
+Wire Wire Line
+	3450 6550 3450 6700
+Text GLabel 3450 6050 1    60   Input ~ 0
++3V3
+Wire Wire Line
+	3450 6250 3450 6050
+$Comp
+L POT R4
+U 1 1 58713E15
+P 4500 6400
+F 0 "R4" H 4430 6446 50  0000 R CNN
+F 1 "10Kb" H 4430 6355 50  0000 R CNN
+F 2 "" H 4500 6400 50  0000 C CNN
+F 3 "" H 4500 6400 50  0000 C CNN
+	1    4500 6400
+	1    0    0    -1
+$EndComp
+Text GLabel 4800 6400 2    60   Input ~ 0
+Pot_4
+Wire Wire Line
+	4800 6400 4650 6400
+$Comp
+L Earth #PWR?
+U 1 1 58713E1D
+P 4500 6700
+F 0 "#PWR?" H 4500 6450 50  0001 C CNN
+F 1 "Earth" H 4500 6550 50  0001 C CNN
+F 2 "" H 4500 6700 50  0000 C CNN
+F 3 "" H 4500 6700 50  0000 C CNN
+	1    4500 6700
+	1    0    0    -1
+$EndComp
+Wire Wire Line
+	4500 6550 4500 6700
+Text GLabel 4500 6050 1    60   Input ~ 0
++3V3
+Wire Wire Line
+	4500 6250 4500 6050
 $EndSCHEMATC
