File: PCB/Estebquencer/Estebquencer.sch (KiCad schematic (older format))
At the start: 6 parts, among them IC1 STM32F103C8T6, IC2 DAC7513_DCN

Commit message: se cambió el DAC del proyecto kicad
Parts:
- removed IC2: DAC7513_DCN, symbol DAC7513_DCN
- added U?: DAC8552, symbol DAC8552
Connections:
- net labels removed: Audio_Out
- wire segments 16 -> 12
Changed lines of the file:
@@
 LIBS:libreria_proyecto
 LIBS:Estebquencer-cache
-EELAYER 26 0
+EELAYER 25 0
 EELAYER END
 $Descr A4 11693 8268
@@
 	1    0    0    -1
 $EndComp
-$Comp
-L DAC7513_DCN IC2
-U 1 1 5871366C
-P 9350 1500
-F 0 "IC2" H 9350 2178 50  0000 C CNN
-F 1 "DAC7513_DCN" H 9350 2087 50  0000 C CNN
-F 2 "" H 9400 1100 50  0000 L CNN
-F 3 "" H 9350 1500 50  0000 C CNN
-	1    9350 1500
-	1    0    0    -1
-$EndComp
-Text GLabel 10450 1300 2    60   Input ~ 0
-Audio_Out
-Wire Wire Line
-	9950 1300 10250 1300
-Wire Wire Line
-	10250 1300 10450 1300
-Wire Wire Line
-	9950 1500 10250 1500
-Wire Wire Line
-	10250 1500 10250 1300
-Connection ~ 10250 1300
 $Comp
 L POT R1
@@
 Wire Wire Line
 	4500 6250 4500 6050
+$Comp
+L DAC8552 U?
+U 1 1 58714820
+P 9100 1650
+F 0 "U?" H 8900 1900 60  0000 C CNN
+F 1 "DAC8552" H 8950 1400 60  0000 C CNN
+F 2 "" H 9100 1750 60  0001 C CNN
+F 3 "" H 9100 1750 60  0001 C CNN
+	1    9100 1650
+	1    0    0    -1
+$EndComp
 $EndSCHEMATC

Commit message: cristal nuevo
Parts:
- added C1, C2: 18p, symbol CP1
- added Q1: 8Mhz, symbol Crystal
Connections:
- wire segments 12 -> 27
Changed lines of the file:
@@
 LIBS:libreria_proyecto
 LIBS:Estebquencer-cache
-EELAYER 25 0
+EELAYER 26 0
 EELAYER END
 $Descr A4 11693 8268
@@
 Text GLabel 1650 6400 2    60   Input ~ 0
 Pot_1
-Wire Wire Line
-	1650 6400 1500 6400
 $Comp
 L Earth #PWR?
@@
 	1    0    0    -1
 $EndComp
-Wire Wire Line
-	1350 6550 1350 6700
 Text GLabel 1350 6050 1    60   Input ~ 0
 +3V3
-Wire Wire Line
-	1350 6250 1350 6050
 $Comp
 L POT R2
@@
 Text GLabel 2700 6400 2    60   Input ~ 0
 Pot_2
-Wire Wire Line
-	2700 6400 2550 6400
 $Comp
 L Earth #PWR?
@@
 	1    0    0    -1
 $EndComp
-Wire Wire Line
-	2400 6550 2400 6700
 Text GLabel 2400 6050 1    60   Input ~ 0
 +3V3
-Wire Wire Line
-	2400 6250 2400 6050
 $Comp
 L POT R3
@@
 Text GLabel 3750 6400 2    60   Input ~ 0
 Pot_3
-Wire Wire Line
-	3750 6400 3600 6400
 $Comp
 L Earth #PWR?
@@
 	1    0    0    -1
 $EndComp
-Wire Wire Line
-	3450 6550 3450 6700
 Text GLabel 3450 6050 1    60   Input ~ 0
 +3V3
-Wire Wire Line
-	3450 6250 3450 6050
 $Comp
 L POT R4
@@
 Text GLabel 4800 6400 2    60   Input ~ 0
 Pot_4
-Wire Wire Line
-	4800 6400 4650 6400
 $Comp
 L Earth #PWR?
@@
 	1    0    0    -1
 $EndComp
-Wire Wire Line
-	4500 6550 4500 6700
 Text GLabel 4500 6050 1    60   Input ~ 0
 +3V3
-Wire Wire Line
-	4500 6250 4500 6050
 $Comp
 L DAC8552 U?
@@
 	1    0    0    -1
 $EndComp
+$Comp
+L Crystal Q1
+U 1 1 587155DF
+P 1300 2200
+F 0 "Q1" V 1346 2069 50  0000 R CNN
+F 1 "8Mhz" V 1255 2069 50  0000 R CNN
+F 2 "" H 1300 2200 50  0000 C CNN
+F 3 "" H 1300 2200 50  0000 C CNN
+	1    1300 2200
+	0    -1   -1   0
+$EndComp
+$Comp
+L CP1 C1
+U 1 1 58715A1B
+P 1100 2550
+F 0 "C1" V 1352 2550 50  0000 C CNN
+F 1 "18p" V 1261 2550 50  0000 C CNN
+F 2 "" H 1100 2550 50  0000 C CNN
+F 3 "" H 1100 2550 50  0000 C CNN
+	1    1100 2550
+	0    -1   -1   0
+$EndComp
+$Comp
+L CP1 C2
+U 1 1 58715AD3
+P 1100 1900
+F 0 "C2" V 1352 1900 50  0000 C CNN
+F 1 "18p" V 1261 1900 50  0000 C CNN
+F 2 "" H 1100 1900 50  0000 C CNN
+F 3 "" H 1100 1900 50  0000 C CNN
+	1    1100 1900
+	0    -1   -1   0
+$EndComp
+Wire Wire Line
+	1650 6400 1500 6400
+Wire Wire Line
+	1350 6550 1350 6700
+Wire Wire Line
+	1350 6250 1350 6050
+Wire Wire Line
+	2700 6400 2550 6400
+Wire Wire Line
+	2400 6550 2400 6700
+Wire Wire Line
+	2400 6250 2400 6050
+Wire Wire Line
+	3750 6400 3600 6400
+Wire Wire Line
+	3450 6550 3450 6700
+Wire Wire Line
+	3450 6250 3450 6050
+Wire Wire Line
+	4800 6400 4650 6400
+Wire Wire Line
+	4500 6550 4500 6700
+Wire Wire Line
+	4500 6250 4500 6050
+Wire Wire Line
+	1250 2550 1300 2550
+Wire Wire Line
+	1300 2550 1300 2350
+Wire Wire Line
+	1850 2250 1700 2250
+Wire Wire Line
+	1700 2250 1700 2400
+Wire Wire Line
+	1700 2400 1300 2400
+Connection ~ 1300 2400
+Wire Wire Line
+	1850 2150 1700 2150
+Wire Wire Line
+	1700 2150 1700 2000
+Wire Wire Line
+	1700 2000 1300 2000
+Wire Wire Line
+	1300 1900 1300 2050
+Wire Wire Line
+	1300 1900 1250 1900
+Connection ~ 1300 2000
+Wire Wire Line
+	950  1900 850  1900
+Wire Wire Line
+	850  1900 850  2550
+Wire Wire Line
+	850  2550 950  2550
+$Comp
+L Earth #PWR?
+U 1 1 58715C9E
+P 650 2400
+F 0 "#PWR?" H 650 2150 50  0001 C CNN
+F 1 "Earth" H 650 2250 50  0001 C CNN
+F 2 "" H 650 2400 50  0000 C CNN
+F 3 "" H 650 2400 50  0000 C CNN
+	1    650  2400
+	1    0    0    -1
+$EndComp
+Connection ~ 850  2250
+Wire Wire Line
+	850  2250 650  2250
+Wire Wire Line
+	650  2250 650  2400
 $EndSCHEMATC

Commit message: cambios en el proyecto kicad de forma temporal, hojas jerárquicas para mostrar su funcionamiento
Connections:
- wire segments 27 -> 35
Other:
- note added: "haz click derecho dentro del cuadradito\ny después en " enter sheet "\n(también vale doble click)"
Changed lines of the file:
@@
 LIBS:libreria_proyecto
 LIBS:Estebquencer-cache
-EELAYER 26 0
+EELAYER 25 0
 EELAYER END
 $Descr A4 11693 8268
 encoding utf-8
-Sheet 1 1
+Sheet 1 2
 Title ""
 Date ""
@@
 Wire Wire Line
 	650  2250 650  2400
+$Sheet
+S 8900 4300 700  600
+U 58715979
+F0 "Operacional" 60
+F1 "test_operacional.sch" 60
+F2 "input" I L 8900 4550 60
+F3 "output" I R 9600 4550 60
+$EndSheet
+Text Notes 8700 4100 0    60   ~ 0
+haz click derecho dentro del cuadradito\ny después en " enter sheet "\n(también vale doble click)
+Wire Wire Line
+	8900 4550 8550 4550
+Wire Wire Line
+	8550 4550 8550 4250
+Wire Wire Line
+	8550 4250 7650 4250
+Wire Wire Line
+	7650 4350 8350 4350
+Wire Wire Line
+	8350 4350 8350 5150
+Wire Wire Line
+	8350 5150 10200 5150
+Wire Wire Line
+	10200 5150 10200 4550
+Wire Wire Line
+	10200 4550 9600 4550
 $EndSCHEMATC

Commit message: cambios en el proyecto kicad de forma temporal, hojas jerárquicas para mostrar su funcionamiento
Parts:
- added IC?: AT89C2051-P, DIP20, symbol AT89C2051-P
Other:
- moved on the sheet: U?
Changed lines of the file:
@@
 L DAC8552 U?
 U 1 1 58714820
-P 9100 1650
-F 0 "U?" H 8900 1900 60  0000 C CNN
-F 1 "DAC8552" H 8950 1400 60  0000 C CNN
-F 2 "" H 9100 1750 60  0001 C CNN
-F 3 "" H 9100 1750 60  0001 C CNN
-	1    9100 1650
+P 8550 850
+F 0 "U?" H 8350 1100 60  0000 C CNN
+F 1 "DAC8552" H 8400 600 60  0000 C CNN
+F 2 "" H 8550 950 60  0001 C CNN
+F 3 "" H 8550 950 60  0001 C CNN
+	1    8550 850
 	1    0    0    -1
 $EndComp
@@
 Wire Wire Line
 	10200 4550 9600 4550
+$Comp
+L AT89C2051-P IC?
+U 1 1 58715DCF
+P 9900 2550
+F 0 "IC?" H 8950 3550 50  0000 C CNN
+F 1 "AT89C2051-P" H 10650 1650 50  0000 C CNN
+F 2 "DIP20" H 9900 2550 50  0000 C CIN
+F 3 "" H 9900 2550 50  0000 C CNN
+	1    9900 2550
+	1    0    0    -1
+$EndComp
 $EndSCHEMATC

Commit message: asd
Parts:
- removed IC?: AT89C2051-P, DIP20, symbol AT89C2051-P
- added IC2, IC3, IC?: 74HC595, symbol 74HC595
- R1, R2, R3, R4: symbol POT -> POT-RESCUE-Estebquencer
- gave numbers to parts that had none: 1
- renumbered IC1 to UC1
Connections:
- net labels added: Audio_out_, Audio_out_osc, DISP_CHAR0, DISP_CHAR1, DISP_CHAR2, DISP_CHAR3, DISP_EN, DISP_SCK, DISP_SER, Decay_out, Env_Mod_out, Pot_1_Tunning, Pot_2_Decay, Pot_3_Env_Mod, Pot_4_Accent
- net labels removed: Pot_1, Pot_2, Pot_3, Pot_4
- wire segments 35 -> 73
Other:
- note removed: "haz click derecho dentro del cuadradito\ny después en " enter sheet "\n(también vale doble click)"
- moved on the sheet: IC1, R1, R2, R3, R4

Commit message: Se recuperó la librería_local, se hizo la hoja del kicad más grande, se creó el componente ACPSC04-41SURKWA, se añadió el datasheet del ACPSC04-41SURKWA.
Parts:
- added U? (x2): ACPSC04-41SURKWA, symbol ACPSC04-41SURKWA
Other:
- moved on the sheet: C1, C2, IC1, IC2, IC3, IC?, Q1, R1, R2, R3, R4, UC1

Commit message: “minor”
Parts:
- added P? (x2): DIN_5, symbol DIN_5
- added Q1, Q2, Q3, Q4: MMBT3904, SOT-23, symbol MMBT3904
- added R1, R2, R3, R4: 1.0K, symbol R
- added SW1: Rotary_Encoder_Switch, symbol Rotary_Encoder_Switch
Connections:
- net +3V3: no longer R1.1
- net DISP_CHAR0: now also R1.2
- net DISP_CHAR1: now also R2.2
- net DISP_CHAR2: now also R3.2
- net DISP_CHAR3: now also R4.2
- net Earth: now also UC1.2 (PC13/RTC_OUT/RTC_TAMPER), UC1.3 (PC14/RCC_OSC32_IN), UC1.4 (PC15/ADC1_EXTI15/ADC2_EXTI15/RCC_OSC32_OUT), Q1.2 (E), Q2.2 (E), Q3.2 (E), Q4.2 (E), SW1.1 (A), SW1.3 (B), SW1.4, SW1.5
- net Gate_A: now reaches UC1.18 (PB0/ADC1_IN8/ADC2_IN8/TIM1_CH2N/TIM3_CH3)
- net at U?.11 (B): now also Q2.3 (C)
- net at U?.16 (F): now also Q1.3 (C)
- net at U?.11 (B): now also Q4.3 (C)
- net at U?.16 (F): now also Q3.3 (C)
- new net: Q4.1 (B), R4.1
- new net: Q3.1 (B), R3.1
- new net: Q2.1 (B), R2.1
- new net: Q1.1 (B), R1.1
Other:
- moved on the sheet: C1, C2, IC1, IC2, IC3, IC?, Q1, R1, R2, R3, R4, U?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

Commit message: Se añadió hoja de medidas en la carpeta Dibujos. Se limpió el esquemático. Se terminó: bloque display, DAC, Encoder y potes.
Parts:
- removed C1, C2: 18p, symbol CP1
- removed IC1: DAC8552, symbol DAC8552
- removed IC2, IC3, IC?: 74HC595, symbol 74HC595
- removed P? (x2): DIN_5, symbol DIN_5
- removed Q1: 8Mhz, symbol Crystal
- removed Q1, Q2, Q3, Q4: MMBT3904, SOT-23, symbol MMBT3904
- removed R1, R2, R3, R4: 10Kb, symbol POT-RESCUE-Estebquencer
- removed R1, R2, R3, R4: 1.0K, symbol R
- removed SW1: Rotary_Encoder_Switch, symbol Rotary_Encoder_Switch
- removed U? (x2): ACPSC04-41SURKWA, symbol ACPSC04-41SURKWA
- removed UC1: STM32F103C8T6, LQFP48, symbol STM32F103C8T6
Other:
- note added: "Falta:"
- note added: "Notas:"
- note added: "·ARM"
- note added: "·JTAG"
- note added: "·MIDI"
- note added: "·Módulo DAC terminado. No tocar"
- note added: "·Módulo Encoder terminado. No tocar"
- note added: "·Módulo Potes terminado. No tocar"
- note added: "·Módulo display terminado. No tocar"
