File: PCB/Estebquencer/HT16K33.sch (KiCad schematic (older format))
At the start: 4 parts

Commit message: Había un pin desconectador de la matriz de LEDs
Parts:
- gave numbers to parts that had none: 4
Changed lines of the file:
@@
 C7
 $Comp
-L libreria_proyecto:HT16K33 U?
+L libreria_proyecto:HT16K33 U4
 U 1 1 5EB7B8AB
 P 5600 4250
-F 0 "U?" H 5575 5041 60  0000 C CNN
+F 0 "U4" H 5575 5041 60  0000 C CNN
 F 1 "HT16K33" H 5700 3500 60  0001 C CNN
 F 2 "" H 5400 4850 60  0001 C CNN
@@
 $EndComp
 $Comp
-L Device:C_Small C?
+L Device:C_Small C7
 U 1 1 5EB803CA
 P 4900 6950
-F 0 "C?" H 4992 6996 50  0000 L CNN
+F 0 "C7" H 4992 6996 50  0000 L CNN
 F 1 "100nF" H 4992 6905 50  0000 L CNN
 F 2 "" H 4900 6950 50  0001 C CNN
@@
 $EndComp
 $Comp
-L Device:R_Small R?
+L Device:R_Small R15
 U 1 1 5EB8328E
 P 6400 3550
-F 0 "R?" V 6500 3550 50  0000 C CNN
+F 0 "R15" V 6500 3550 50  0000 C CNN
 F 1 "4.7K" V 6400 3550 50  0000 C CNN
 F 2 "" H 6400 3550 50  0001 C CNN
@@
 $EndComp
 $Comp
-L Device:R_Small R?
+L Device:R_Small R16
 U 1 1 5EB833FD
 P 6500 3550
-F 0 "R?" V 6400 3550 50  0000 C CNN
+F 0 "R16" V 6400 3550 50  0000 C CNN
 F 1 "4.7K" V 6500 3550 50  0000 C CNN
 F 2 "" H 6500 3550 50  0001 C CNN
@@
 Wire Wire Line
 	6500 3400 6500 3350
-Wire Wire Line
-	6200 3350 6200 3600
 Wire Wire Line
 	6100 3700 6400 3700
@@
 Wire Wire Line
 	5050 4500 4950 4500
+Wire Wire Line
+	6200 3600 6200 3350
 $EndSCHEMATC
