File: PCB/Estebquencer/JTAG.sch (KiCad schematic (older format))
At the start: 0 parts

Commit message: se cablearon los módulos al ARM, se añadió el conector JTAG (SWD)
Parts:
- added P?: CONN_01X03, symbol CONN_01X03
Connections:
- new net GNDREF: P?.3 (P3)
- new net SWCLK: P?.2 (P2)
- new net SWDIO: P?.1 (P1)
Changed lines of the file:
@@
 EELAYER 25 0
 EELAYER END
-$Descr A4 11693 8268
+$Descr User 5937 4000
 encoding utf-8
-Sheet 1 9
+Sheet 8 9
 Title ""
 Date ""
@@
 Comment4 ""
 $EndDescr
+$Comp
+L CONN_01X03 P?
+U 1 1 587395E4
+P 3200 1500
+F 0 "P?" H 3200 1700 50  0000 C CNN
+F 1 "CONN_01X03" V 3300 1500 50  0000 C CNN
+F 2 "" H 3200 1500 50  0000 C CNN
+F 3 "" H 3200 1500 50  0000 C CNN
+	1    3200 1500
+	1    0    0    -1
+$EndComp
+$Comp
+L GNDREF #PWR?
+U 1 1 58739785
+P 2850 1750
+F 0 "#PWR?" H 2850 1500 50  0001 C CNN
+F 1 "GNDREF" H 2850 1600 50  0000 C CNN
+F 2 "" H 2850 1750 50  0000 C CNN
+F 3 "" H 2850 1750 50  0000 C CNN
+	1    2850 1750
+	1    0    0    -1
+$EndComp
+Wire Wire Line
+	3000 1600 2850 1600
+Wire Wire Line
+	2850 1600 2850 1750
+Text HLabel 2800 1400 0    60   Input ~ 0
+SWDIO
+Text HLabel 2800 1500 0    60   Input ~ 0
+SWCLK
+Wire Wire Line
+	2800 1500 3000 1500
+Wire Wire Line
+	3000 1400 2800 1400
 $EndSCHEMATC

Commit message: Añadido proyecto ST, configuración superficial de todos los periféricos, falta crear los threads en FreeRTOS
Parts:
- P?: symbol CONN_01X03 -> Estebquencer-rescue:CONN_01X03
Changed lines of the file:
@@
-EESchema Schematic File Version 2
-LIBS:libreria_proyecto
-LIBS:74xgxx
-LIBS:74xx
-LIBS:ac-dc
-LIBS:actel
-LIBS:adc-dac
-LIBS:Altera
-LIBS:analog_devices
-LIBS:analog_switches
-LIBS:atmel
-LIBS:audio
-LIBS:brooktre
-LIBS:cmos4000
-LIBS:cmos_ieee
-LIBS:conn
-LIBS:contrib
-LIBS:cypress
-LIBS:dc-dc
-LIBS:device
-LIBS:digital-audio
-LIBS:diode
-LIBS:display
-LIBS:dsp
-LIBS:elec-unifil
-LIBS:ESD_Protection
-LIBS:ftdi
-LIBS:gennum
-LIBS:graphic
-LIBS:hc11
-LIBS:intel
-LIBS:interface
-LIBS:ir
-LIBS:Lattice
-LIBS:linear
-LIBS:logo
-LIBS:maxim
-LIBS:memory
-LIBS:microchip
-LIBS:microchip_dspic33dsc
-LIBS:microchip_pic10mcu
-LIBS:microchip_pic12mcu
-LIBS:microchip_pic16mcu
-LIBS:microchip_pic18mcu
-LIBS:microchip_pic32mcu
-LIBS:microcontrollers
-LIBS:motor_drivers
-LIBS:motorola
-LIBS:msp430
-LIBS:nordicsemi
-LIBS:nxp_armmcu
-LIBS:onsemi
-LIBS:opto
-LIBS:Oscillators
-LIBS:philips
-LIBS:power
-LIBS:powerint
-LIBS:Power_Management
-LIBS:pspice
-LIBS:references
-LIBS:regul
-LIBS:relays
-LIBS:rfcom
-LIBS:sensors
-LIBS:silabs
-LIBS:siliconi
-LIBS:stm8
-LIBS:stm32
-LIBS:supertex
-LIBS:switches
-LIBS:texas
-LIBS:transf
-LIBS:transistors
-LIBS:ttl_ieee
-LIBS:valves
-LIBS:video
-LIBS:Xicor
-LIBS:xilinx
-LIBS:Zilog
+EESchema Schematic File Version 4
 LIBS:Estebquencer-cache
-EELAYER 25 0
+EELAYER 26 0
 EELAYER END
 $Descr User 5937 4000
 encoding utf-8
-Sheet 8 9
+Sheet 8 10
 Title ""
 Date ""
@@
 $EndDescr
 $Comp
-L CONN_01X03 P?
+L Estebquencer-rescue:CONN_01X03 P?
 U 1 1 587395E4
 P 3200 1500
@@
 $EndComp
 $Comp
-L GNDREF #PWR?
+L power:GNDREF #PWR?
 U 1 1 58739785
 P 2850 1750

Commit message: acabado módulo ARM
Connections:
- net GNDREF renamed GND
Changed lines of the file:
@@
-	1    0    0    -1
-$EndComp
-$Comp
-L power:GNDREF #PWR?
-U 1 1 58739785
-P 2850 1750
-F 0 "#PWR?" H 2850 1500 50  0001 C CNN
-F 1 "GNDREF" H 2850 1600 50  0000 C CNN
-F 2 "" H 2850 1750 50  0000 C CNN
-F 3 "" H 2850 1750 50  0000 C CNN
-	1    2850 1750
 	1    0    0    -1
 $EndComp
@@
 Wire Wire Line
 	3000 1400 2800 1400
+$Comp
+L power:GND #PWR?
+U 1 1 5E3C88E2
+P 2850 1750
+F 0 "#PWR?" H 2850 1500 50  0001 C CNN
+F 1 "GND" H 2855 1577 50  0000 C CNN
+F 2 "" H 2850 1750 50  0001 C CNN
+F 3 "" H 2850 1750 50  0001 C CNN
+	1    2850 1750
+	1    0    0    -1
+$EndComp
 $EndSCHEMATC

Commit message: Había un pin desconectador de la matriz de LEDs
Parts:
- gave numbers to parts that had none: 1
Changed lines of the file:
@@
 $EndDescr
 $Comp
-L Estebquencer-rescue:CONN_01X03 P?
+L Estebquencer-rescue:CONN_01X03 P1
 U 1 1 587395E4
 P 3200 1500
-F 0 "P?" H 3200 1700 50  0000 C CNN
+F 0 "P1" H 3200 1700 50  0000 C CNN
 F 1 "CONN_01X03" V 3300 1500 50  0000 C CNN
-F 2 "" H 3200 1500 50  0000 C CNN
+F 2 "" H 3200 1500 50  0001 C CNN
 F 3 "" H 3200 1500 50  0000 C CNN
 	1    3200 1500
