File: PCB/Estebquencer/arm.sch (KiCad schematic (older format))
At the start: 10 parts

Commit message: Se tuvo que cambiar el sistema de gestión de los LED y pulsadores. Con el charlieplexing no tenía los resultados esperados, así que se le añadió un HT16K33 para hacer las cosas más simples y fluídas. También se usará el mismo IC para la gestión de botones, ya que da opción.
Connections:
- net Btn_C1: no longer names the net of U?.46 (PB9/CAN_TX/I2C1_SDA/TIM4_CH4)
- net Btn_C2: no longer names the net of U?.45 (PB8/CAN_RX/I2C1_SCL/TIM4_CH3)
- net Btn_C3 renamed HT16K33_SDA
- net Btn_C4 renamed HT16K33_SCL
- net Btn_C5 renamed HT16K33_INT
- net Btn_C6: no longer names the net of U?.40 (PB4/SPI1_MISO/SYS_NJTRST/TIM3_CH1)
- net Btn_C7: no longer names the net of U?.39 (PB3/SPI1_SCK/SYS_JTDO-TRACESWO/TIM2_CH2)
- net Btn_R1: no longer names the net of U?.2 (PC13/RTC_OUT/RTC_TAMPER)
- net Btn_R2: no longer names the net of U?.3 (PC14/RCC_OSC32_IN)
- net Btn_R3: no longer names the net of U?.4 (PC15/ADC1_EXTI15/ADC2_EXTI15/RCC_OSC32_OUT)
- net LED_R1: no longer names the net of U?.31 (TIM1_CH3/USART1_RX/PA10)
- net LED_R2: no longer names the net of U?.30 (TIM1_CH2/USART1_TX/PA9)
- net LED_R3: no longer names the net of U?.29 (RCC_MCO/TIM1_CH1/USART1_CK/PA8)
- net LED_R4: no longer names the net of U?.28 (PB15/ADC1_EXTI15/ADC2_EXTI15/SPI2_MOSI/TIM1_CH3N)
- net LED_R5: no longer names the net of U?.27 (PB14/SPI2_MISO/TIM1_CH2N/USART3_RTS)
- net LED_R6: no longer names the net of U?.26 (PB13/SPI2_SCK/TIM1_CH1N/USART3_CTS)
- net LED_R7: no longer names the net of U?.25 (PB12/I2C2_SMBA/SPI2_NSS/TIM1_BKIN/USART3_CK)
- no-connect marks 4 -> 18
Changed lines of the file:
@@
 $Descr A4 11693 8268
 encoding utf-8
-Sheet 6 10
+Sheet 8 11
 Title ""
 Date ""
@@
 Connection ~ 6200 5400
 $Comp
-L power:+3.3V #PWR?
+L power:+3.3V #PWR0114
 U 1 1 5875F531
 P 6100 1500
-F 0 "#PWR?" H 6100 1350 50  0001 C CNN
+F 0 "#PWR0114" H 6100 1350 50  0001 C CNN
 F 1 "+3.3V" H 6100 1640 50  0000 C CNN
 F 2 "" H 6100 1500 50  0000 C CNN
@@
 Wire Wire Line
 	9200 3700 9400 3700
-Text HLabel 3300 4300 0    60   Input ~ 0
-Btn_C1
-Text HLabel 3300 4200 0    60   Input ~ 0
-Btn_C2
-Text HLabel 3300 4100 0    60   Input ~ 0
-Btn_C3
-Text HLabel 3300 4000 0    60   Input ~ 0
-Btn_C4
-Text HLabel 3300 3900 0    60   Input ~ 0
-Btn_C5
-Text HLabel 3300 3800 0    60   Input ~ 0
-Btn_C6
-Text HLabel 3300 3700 0    60   Input ~ 0
-Btn_C7
-Wire Wire Line
-	3400 4300 3300 4300
-Wire Wire Line
-	3300 4200 3400 4200
-Wire Wire Line
-	3400 4100 3300 4100
-Wire Wire Line
-	3300 4000 3400 4000
-Wire Wire Line
-	3400 3900 3300 3900
-Wire Wire Line
-	3300 3800 3400 3800
-Wire Wire Line
-	3400 3700 3300 3700
-Text HLabel 3300 3000 0    60   Input ~ 0
-Btn_R1
-Text HLabel 3300 3100 0    60   Input ~ 0
-Btn_R2
-Text HLabel 3300 3200 0    60   Input ~ 0
-Btn_R3
-Wire Wire Line
-	3300 3200 3400 3200
-Wire Wire Line
-	3400 3100 3300 3100
-Wire Wire Line
-	3300 3000 3400 3000
 Text HLabel 9400 3800 2    60   Input ~ 0
 CLK_OUT_2
@@
 Wire Wire Line
 	3300 3400 3400 3400
-Text HLabel 9400 4400 2    60   Input ~ 0
-LED_R1
-Text HLabel 9400 4300 2    60   Input ~ 0
-LED_R2
-Text HLabel 9400 4200 2    60   Input ~ 0
-LED_R3
 Text HLabel 9400 4500 2    60   Input ~ 0
 USB_D-
@@
 Wire Wire Line
 	9200 4500 9400 4500
-Wire Wire Line
-	9400 4400 9200 4400
-Wire Wire Line
-	9200 4300 9400 4300
-Wire Wire Line
-	9400 4200 9200 4200
-Text HLabel 3300 4900 0    60   Input ~ 0
-LED_R4
-Wire Wire Line
-	3300 4900 3400 4900
-Text HLabel 3300 4800 0    60   Input ~ 0
-LED_R5
-Text HLabel 3300 4700 0    60   Input ~ 0
-LED_R6
-Text HLabel 3300 4600 0    60   Input ~ 0
-LED_R7
-Wire Wire Line
-	3300 4600 3400 4600
-Wire Wire Line
-	3400 4700 3300 4700
-Wire Wire Line
-	3300 4800 3400 4800
 Wire Wire Line
 	9200 4900 9400 4900
@@
 $EndComp
 $Comp
-L power:GND #PWR?
+L power:GND #PWR0115
 U 1 1 5E3C872F
 P 6100 5550
-F 0 "#PWR?" H 6100 5300 50  0001 C CNN
+F 0 "#PWR0115" H 6100 5300 50  0001 C CNN
 F 1 "GND" H 6105 5377 50  0000 C CNN
 F 2 "" H 6100 5550 50  0001 C CNN
@@
 $EndComp
 $Comp
-L power:GND #PWR?
+L power:GND #PWR0116
 U 1 1 5E3CBE0D
 P 3300 7350
-F 0 "#PWR?" H 3300 7100 50  0001 C CNN
+F 0 "#PWR0116" H 3300 7100 50  0001 C CNN
 F 1 "GND" H 3305 7177 50  0000 C CNN
 F 2 "" H 3300 7350 50  0001 C CNN
@@
 $EndComp
 $Comp
-L power:+3.3V #PWR?
+L power:+3.3V #PWR0117
 U 1 1 5E3CBE42
 P 3300 6950
-F 0 "#PWR?" H 3300 6800 50  0001 C CNN
+F 0 "#PWR0117" H 3300 6800 50  0001 C CNN
 F 1 "+3.3V" H 3300 7090 50  0000 C CNN
 F 2 "" H 3300 6950 50  0000 C CNN
@@
 $EndComp
 $Comp
-L power:+3.3V #PWR?
+L power:+3.3V #PWR0118
 U 1 1 5E3CBE88
 P 3050 6950
-F 0 "#PWR?" H 3050 6800 50  0001 C CNN
+F 0 "#PWR0118" H 3050 6800 50  0001 C CNN
 F 1 "+3.3V" H 3050 7090 50  0000 C CNN
 F 2 "" H 3050 6950 50  0000 C CNN
@@
 $EndComp
 $Comp
-L power:GND #PWR?
+L power:GND #PWR0119
 U 1 1 5E3CBEC9
 P 3050 7350
-F 0 "#PWR?" H 3050 7100 50  0001 C CNN
+F 0 "#PWR0119" H 3050 7100 50  0001 C CNN
 F 1 "GND" H 3055 7177 50  0000 C CNN
 F 2 "" H 3050 7350 50  0001 C CNN
@@
 $EndComp
 $Comp
-L power:GND #PWR?
+L power:GND #PWR0120
 U 1 1 5E3D0FFF
 P 4050 7350
-F 0 "#PWR?" H 4050 7100 50  0001 C CNN
+F 0 "#PWR0120" H 4050 7100 50  0001 C CNN
 F 1 "GND" H 4055 7177 50  0000 C CNN
 F 2 "" H 4050 7350 50  0001 C CNN
@@
 $EndComp
 $Comp
-L power:+3.3V #PWR?
+L power:+3.3V #PWR0121
 U 1 1 5E3D1005
 P 4050 6950
-F 0 "#PWR?" H 4050 6800 50  0001 C CNN
+F 0 "#PWR0121" H 4050 6800 50  0001 C CNN
 F 1 "+3.3V" H 4050 7090 50  0000 C CNN
 F 2 "" H 4050 6950 50  0000 C CNN
@@
 $EndComp
 $Comp
-L power:+3.3V #PWR?
+L power:+3.3V #PWR0122
 U 1 1 5E3D100B
 P 3800 6950
-F 0 "#PWR?" H 3800 6800 50  0001 C CNN
+F 0 "#PWR0122" H 3800 6800 50  0001 C CNN
 F 1 "+3.3V" H 3800 7090 50  0000 C CNN
 F 2 "" H 3800 6950 50  0000 C CNN
@@
 $EndComp
 $Comp
-L power:GND #PWR?
+L power:GND #PWR0123
 U 1 1 5E3D1011
 P 3800 7350
-F 0 "#PWR?" H 3800 7100 50  0001 C CNN
+F 0 "#PWR0123" H 3800 7100 50  0001 C CNN
 F 1 "GND" H 3805 7177 50  0000 C CNN
 F 2 "" H 3800 7350 50  0001 C CNN
@@
 Boot_0
 $Comp
-L power:+3.3V #PWR?
+L power:+3.3V #PWR0124
 U 1 1 5E3C024D
 P 4850 6750
-F 0 "#PWR?" H 4850 6600 50  0001 C CNN
+F 0 "#PWR0124" H 4850 6600 50  0001 C CNN
 F 1 "+3.3V" H 4850 6890 50  0000 C CNN
 F 2 "" H 4850 6750 50  0000 C CNN
@@
 $EndComp
 $Comp
-L power:GND #PWR?
+L power:GND #PWR0125
 U 1 1 5E3C0266
 P 4850 7350
-F 0 "#PWR?" H 4850 7100 50  0001 C CNN
+F 0 "#PWR0125" H 4850 7100 50  0001 C CNN
 F 1 "GND" H 4855 7177 50  0000 C CNN
 F 2 "" H 4850 7350 50  0001 C CNN
@@
 Connection ~ 5600 7000
 $Comp
-L power:GND #PWR?
+L power:GND #PWR0126
 U 1 1 5E3D0E6F
 P 5600 7350
-F 0 "#PWR?" H 5600 7100 50  0001 C CNN
+F 0 "#PWR0126" H 5600 7100 50  0001 C CNN
 F 1 "GND" H 5605 7177 50  0000 C CNN
 F 2 "" H 5600 7350 50  0001 C CNN
@@
 	5600 7350 5600 7250
 $Comp
-L power:+3.3V #PWR?
+L power:+3.3V #PWR0127
 U 1 1 5E3D4E71
 P 5600 6600
-F 0 "#PWR?" H 5600 6450 50  0001 C CNN
+F 0 "#PWR0127" H 5600 6450 50  0001 C CNN
 F 1 "+3.3V" H 5600 6740 50  0000 C CNN
 F 2 "" H 5600 6600 50  0000 C CNN
@@
 	6250 6700 6250 6750
 $Comp
-L power:GND #PWR?
+L power:GND #PWR0128
 U 1 1 5E3E61E8
 P 6350 7250
-F 0 "#PWR?" H 6350 7000 50  0001 C CNN
+F 0 "#PWR0128" H 6350 7000 50  0001 C CNN
 F 1 "GND" H 6355 7077 50  0000 C CNN
 F 2 "" H 6350 7250 50  0001 C CNN
@@
 Text Notes 4350 7250 0    60   ~ 0
 -->Flash
+Text HLabel 3300 4100 0    60   Input ~ 0
+HT16K33_SDA
+Text HLabel 3300 4000 0    60   Input ~ 0
+HT16K33_SCL
+Wire Wire Line
+	3300 4000 3400 4000
+Wire Wire Line
+	3400 4100 3300 4100
+Wire Wire Line
+	3400 3700 3300 3700
+Wire Wire Line
+	3300 3800 3400 3800
+Wire Wire Line
+	3400 4600 3300 4600
+Wire Wire Line
+	3300 4700 3400 4700
+Wire Wire Line
+	3300 4800 3400 4800
+Wire Wire Line
+	3300 4900 3400 4900
+Wire Wire Line
+	3300 4200 3400 4200
+Wire Wire Line
+	3300 4300 3400 4300
+Wire Wire Line
+	3400 3000 3300 3000
+Wire Wire Line
+	3300 3100 3400 3100
+Wire Wire Line
+	3300 3200 3400 3200
+Wire Wire Line
+	9400 4300 9200 4300
+Wire Wire Line
+	9200 4200 9400 4200
+Wire Wire Line
+	9400 4400 9200 4400
+NoConn ~ 9400 4400
+NoConn ~ 9400 4300
+NoConn ~ 9400 4200
+NoConn ~ 3300 4900
+NoConn ~ 3300 4800
+NoConn ~ 3300 4700
+NoConn ~ 3300 4600
+NoConn ~ 3300 4300
+NoConn ~ 3300 4200
+NoConn ~ 3300 3800
+NoConn ~ 3300 3700
+NoConn ~ 3300 3200
+NoConn ~ 3300 3100
+NoConn ~ 3300 3000
+Text HLabel 3300 3900 0    60   Input ~ 0
+HT16K33_INT
+Wire Wire Line
+	3300 3900 3400 3900
 $EndSCHEMATC

Commit message: Había un pin desconectador de la matriz de LEDs
Parts:
- gave numbers to parts that had none: 10
Changed lines of the file:
@@
 $EndDescr
 $Comp
-L libreria_proyecto:STM32F103C8T6 U?
+L libreria_proyecto:STM32F103C8T6 U5
 U 1 1 5875A9A5
 P 6300 3500
-F 0 "U?" H 3500 5225 50  0000 L BNN
+F 0 "U5" H 3500 5225 50  0000 L BNN
 F 1 "STM32F103C8T6" H 9100 5225 50  0000 R BNN
 F 2 "LQFP48" H 9100 5175 50  0000 R TNN
@@
 Wire Wire Line
 	6100 1550 6200 1550
-Wire Wire Line
-	6300 1550 6300 1700
 Connection ~ 6200 1550
 $Sheet
@@
 Wire Wire Line
 	6100 1550 6100 1700
-Wire Wire Line
-	6200 1550 6300 1550
 $Sheet
 S 850  5350 550  300
@@
 Wire Wire Line
 	6400 1700 6400 1550
-Wire Wire Line
-	6400 1550 6300 1550
-Connection ~ 6300 1550
-$Comp
-L Device:C_Small C?
+$Comp
+L Device:C_Small C9
 U 1 1 5E3C7F8F
 P 3300 7150
-F 0 "C?" H 3350 7000 50  0000 L CNN
+F 0 "C9" H 3350 7000 50  0000 L CNN
 F 1 "100nF" V 3400 7050 50  0000 L CNN
 F 2 "" H 3300 7150 50  0001 C CNN
@@
 $EndComp
 $Comp
-L Device:C_Small C?
+L Device:C_Small C8
 U 1 1 5E3C867B
 P 3050 7150
-F 0 "C?" H 3100 7000 50  0000 L CNN
+F 0 "C8" H 3100 7000 50  0000 L CNN
 F 1 "100nF" V 3150 7050 50  0000 L CNN
 F 2 "" H 3050 7150 50  0001 C CNN
@@
 	3300 7250 3300 7350
 $Comp
-L Device:C_Small C?
+L Device:C_Small C11
 U 1 1 5E3D0FF3
 P 4050 7150
-F 0 "C?" H 4100 7000 50  0000 L CNN
+F 0 "C11" H 4100 7000 50  0000 L CNN
 F 1 "100nF" V 4150 7050 50  0000 L CNN
 F 2 "" H 4050 7150 50  0001 C CNN
@@
 $EndComp
 $Comp
-L Device:C_Small C?
+L Device:C_Small C10
 U 1 1 5E3D0FF9
 P 3800 7150
-F 0 "C?" H 3850 7000 50  0000 L CNN
+F 0 "C10" H 3850 7000 50  0000 L CNN
 F 1 "100nF" V 3900 7050 50  0000 L CNN
 F 2 "" H 3800 7150 50  0001 C CNN
@@
 To ARM
 $Comp
-L Device:R_Small R?
+L Device:R_Small R17
 U 1 1 5E3B61C6
 P 4850 6900
-F 0 "R?" H 4750 6850 50  0000 C CNN
+F 0 "R17" H 4750 6850 50  0000 C CNN
 F 1 "10K" V 4850 6900 50  0000 C CNN
 F 2 "" H 4850 6900 50  0001 C CNN
@@
 	4250 7600 2900 7600
 $Comp
-L Device:C_Small C?
+L Device:C_Small C12
 U 1 1 5E3CC93E
 P 5600 7150
-F 0 "C?" H 5692 7196 50  0000 L CNN
+F 0 "C12" H 5692 7196 50  0000 L CNN
 F 1 "1uF" H 5692 7105 50  0000 L CNN
 F 2 "" H 5600 7150 50  0001 C CNN
@@
 $EndComp
 $Comp
-L Device:R R?
+L Device:R R19
 U 1 1 5E3CCF90
 P 5600 6800
-F 0 "R?" H 5670 6846 50  0000 L CNN
+F 0 "R19" H 5670 6846 50  0000 L CNN
 F 1 "10K" V 5600 6750 50  0000 L CNN
 F 2 "" V 5530 6800 50  0001 C CNN
@@
 	1    0    0    -1
 $EndComp
-Wire Wire Line
-	5600 6600 5600 6650
-$Comp
-L Switch:SW_Push_Dual SW?
+$Comp
+L Switch:SW_Push_Dual SW22
 U 1 1 5E3DB4C0
 P 6450 6950
-F 0 "SW?" V 6450 7098 50  0000 L CNN
+F 0 "SW22" V 6450 7098 50  0000 L CNN
 F 1 "SW_Push_Dual" H 6450 7144 50  0001 C CNN
 F 2 "" H 6450 7150 50  0001 C CNN
@@
 Connection ~ 6100 1550
 $Comp
-L Device:R_Small R?
+L Device:R_Small R18
 U 1 1 5E403B53
 P 4850 7200
-F 0 "R?" H 4750 7250 50  0000 C CNN
+F 0 "R18" H 4750 7250 50  0000 C CNN
 F 1 "10K" V 4850 7200 50  0000 C CNN
 F 2 "" H 4850 7200 50  0001 C CNN
@@
 	-1   0    0    1
 $EndComp
-Wire Wire Line
-	4850 6800 4850 6750
 Wire Wire Line
 	4850 7350 4850 7300
@@
 Wire Wire Line
 	3300 3900 3400 3900
+Wire Wire Line
+	6200 1550 6300 1550
+Wire Wire Line
+	6300 1700 6300 1550
+Connection ~ 6300 1550
+Wire Wire Line
+	6300 1550 6400 1550
+Wire Wire Line
+	4850 6800 4850 6750
+Wire Wire Line
+	5600 6650 5600 6600
 $EndSCHEMATC
