File: PCB/Estebquencer/drivers.sch (KiCad schematic (older format))
At the start: 2 parts

Commit message: Terminado módulo DAC
Parts:
- added C? (x2): 100uF, symbol Device:CP1_Small
- added C? (x2): 100nF, symbol Device:C_Small
- added L? (x2): 22uH, symbol Device:L_Small
- added R? (x4): 220, symbol Device:R
Connections:
- net +3V3: now also C?.1, C?.1, C?.1, C?.1, L?.1, L?.1; no longer U?.1 (Vdd), U?.1 (Vdd)
- net CV1: now also R?.1; no longer U?.6 (VB)
- net CV2: now also R?.1; no longer U?.6 (VB)
- net GND: now also C?.2, C?.2, C?.2, C?.2
- net Gate1: now also R?.1; no longer U?.8 (VA)
- net Gate2: now also R?.1; no longer U?.8 (VA)
- new net: R?.2, U?.8 (VA) (x2)
- new net: R?.2, U?.6 (VB) (x2)
- new net: L?.2, U?.1 (Vdd) (x2)
Other:
- note added: "Cerca DAC1"
- note added: "Cerca DAC2"

Commit message: Había un pin desconectador de la matriz de LEDs
Parts:
- gave numbers to parts that had none: 12
Changed lines of the file:
@@
 CV2
 $Comp
-L Analog_DAC:MCP4822 U?
+L Analog_DAC:MCP4822 U1
 U 1 1 5E6BF050
 P 5550 2650
-F 0 "U?" H 5550 3228 50  0001 C CNN
+F 0 "U1" H 5550 3228 50  0001 C CNN
 F 1 "MCP4822" H 5550 3137 50  0001 C CNN
 F 2 "" H 6350 2350 50  0001 C CNN
@@
 $EndComp
 $Comp
-L Analog_DAC:MCP4822 U?
+L Analog_DAC:MCP4822 U2
 U 1 1 5E6BF0E6
 P 5550 4600
-F 0 "U?" H 5550 5086 50  0001 C CNN
+F 0 "U2" H 5550 5086 50  0001 C CNN
 F 1 "MCP4822" H 5550 5087 50  0001 C CNN
 F 2 "" H 6350 4300 50  0001 C CNN
@@
 	5550 3200 5550 3250
 $Comp
-L Device:R R?
+L Device:R R1
 U 1 1 5E3B0F09
 P 6300 2550
-F 0 "R?" V 6200 2500 50  0000 C CNN
+F 0 "R1" V 6200 2500 50  0000 C CNN
 F 1 "220" V 6300 2550 50  0000 C CNN
 F 2 "" V 6230 2550 50  0001 C CNN
@@
 	6450 2550 6700 2550
 $Comp
-L Device:R R?
+L Device:R R2
 U 1 1 5E3B1411
 P 6300 2850
-F 0 "R?" V 6400 2800 50  0000 C CNN
+F 0 "R2" V 6400 2800 50  0000 C CNN
 F 1 "220" V 6300 2850 50  0000 C CNN
 F 2 "" V 6230 2850 50  0001 C CNN
@@
 	6450 2850 6700 2850
 $Comp
-L Device:R R?
+L Device:R R3
 U 1 1 5E3B2353
 P 6300 4500
-F 0 "R?" V 6200 4450 50  0000 C CNN
+F 0 "R3" V 6200 4450 50  0000 C CNN
 F 1 "220" V 6300 4500 50  0000 C CNN
 F 2 "" V 6230 4500 50  0001 C CNN
@@
 $EndComp
 $Comp
-L Device:R R?
+L Device:R R4
 U 1 1 5E3B24C4
 P 6300 4800
-F 0 "R?" V 6200 4750 50  0000 C CNN
+F 0 "R4" V 6200 4750 50  0000 C CNN
 F 1 "220" V 6300 4800 50  0000 C CNN
 F 2 "" V 6230 4800 50  0001 C CNN
@@
 $EndComp
 $Comp
-L Device:CP1_Small C?
+L Device:CP1_Small C4
 U 1 1 5E3B4248
 P 4650 6550
-F 0 "C?" H 4700 6650 50  0000 L CNN
+F 0 "C4" H 4700 6650 50  0000 L CNN
 F 1 "100uF" V 4750 6300 50  0000 L CNN
 F 2 "" H 4650 6550 50  0001 C CNN
@@
 $EndComp
 $Comp
-L Device:C_Small C?
+L Device:C_Small C3
 U 1 1 5E3B4321
 P 4400 6550
-F 0 "C?" H 4450 6650 50  0000 L CNN
+F 0 "C3" H 4450 6650 50  0000 L CNN
 F 1 "100nF" V 4500 6350 50  0000 L CNN
 F 2 "" H 4400 6550 50  0001 C CNN
@@
 $EndComp
 $Comp
-L Device:CP1_Small C?
+L Device:CP1_Small C2
 U 1 1 5E3B60D9
 P 3900 6550
-F 0 "C?" H 3950 6650 50  0000 L CNN
+F 0 "C2" H 3950 6650 50  0000 L CNN
 F 1 "100uF" V 4000 6300 50  0000 L CNN
 F 2 "" H 3900 6550 50  0001 C CNN
@@
 $EndComp
 $Comp
-L Device:C_Small C?
+L Device:C_Small C1
 U 1 1 5E3B60DF
 P 3650 6550
-F 0 "C?" H 3700 6650 50  0000 L CNN
+F 0 "C1" H 3700 6650 50  0000 L CNN
 F 1 "100nF" V 3750 6350 50  0000 L CNN
 F 2 "" H 3650 6550 50  0001 C CNN
@@
 Cerca DAC2
 $Comp
-L Device:L_Small L?
+L Device:L_Small L2
 U 1 1 5E3B72FF
 P 5550 4050
-F 0 "L?" H 5598 4096 50  0000 L CNN
+F 0 "L2" H 5598 4096 50  0000 L CNN
 F 1 "22uH" H 5598 4005 50  0000 L CNN
 F 2 "" H 5550 4050 50  0001 C CNN
@@
 Wire Wire Line
 	5550 3900 5550 3950
-Wire Wire Line
-	5550 2200 5550 2250
 $Comp
 L power:+3.3V #PWR0113
@@
 $EndComp
 $Comp
-L Device:L_Small L?
+L Device:L_Small L1
 U 1 1 5E3B7B8C
 P 5550 2100
-F 0 "L?" H 5598 2146 50  0000 L CNN
+F 0 "L1" H 5598 2146 50  0000 L CNN
 F 1 "22uH" H 5598 2055 50  0000 L CNN
 F 2 "" H 5550 2100 50  0001 C CNN
@@
 Wire Wire Line
 	5550 1950 5550 2000
+Wire Wire Line
+	5550 2250 5550 2200
 $EndSCHEMATC
